File: PIC32MX150.sch (KiCad schematic (older format))
At the start: 28 parts, among them J1 GPIO_1, J2 USB_B_Micro, J3 Barrel_Jack, J4 ICSP, J5 GPIO_2, SW1 RST, SW2 SW_SPDT, U1 PIC32MX150F128D-IPT, U2 LM22676MR-ADJ, U3 CH340C

Commit message: LO
Parts:
- added C13, C14: 10p, Capacitor_SMD:C_0603_1608Metric_Pad1.08x0.95mm_HandSolder, symbol Device:C_Small
- added C15: 1u, Capacitor_SMD:C_0603_1608Metric_Pad1.08x0.95mm_HandSolder, symbol Device:C_Small
- added C16, C17, C18: 100n, Capacitor_SMD:C_0603_1608Metric_Pad1.08x0.95mm_HandSolder, symbol Device:C_Small
- added D2, D3: LED_B, LED_SMD:LED_0603_1608Metric_Pad1.05x0.95mm_HandSolder, symbol Device:LED_Small
- added D4: LED_G, LED_SMD:LED_0603_1608Metric_Pad1.05x0.95mm_HandSolder, symbol Device:LED_Small
- added JP1: Jumper_NO_Small, Jumper:SolderJumper-2_P1.3mm_Open_Pad1.0x1.5mm, symbol Device:Jumper_NO_Small
- added R5: 1M, Resistor_SMD:R_0603_1608Metric_Pad0.98x0.95mm_HandSolder, symbol Device:R_Small
- added R6: 1.5K, Resistor_SMD:R_0603_1608Metric_Pad0.98x0.95mm_HandSolder, symbol Device:R_Small
- added R7: 1K, Resistor_SMD:R_0603_1608Metric_Pad0.98x0.95mm_HandSolder, symbol Device:R_Small
- added Y1: TSX3225, Crystal:Crystal_SMD_SeikoEpson_TSX3225-4Pin_3.2x2.5mm_HandSoldering, symbol Device:Crystal_GND24_Small
- J1: footprint Connector_PinHeader_2.54mm:PinHeader_2x12_P2.54mm_Vertical -> Connector_PinSocket_2.54mm:PinSocket_2x12_P2.54mm_Vertical
- L1: footprint Inductor_SMD:L_0805_2012Metric_Pad1.15x1.40mm_HandSolder -> Inductor_SMD:L_Taiyo-Yuden_MD-1616
- SW2: footprint Button_Switch_THT:SW_Slide_1P2T_CK_OS102011MS2Q -> Custom_Libs:SPDT_SW_Big
Connections:
- net +3V3: now also U3.16 (VCC), C17.1, C18.2, D4.2 (A)
- net +5V: now also C15.1, C16.1; no longer U3.16 (VCC)
- net GND: now also U2.5 (EN), C13.2, C14.2, C15.2, C16.2, C17.2, C18.1, R6.2, R7.2, Y1.2, Y1.4
- net PWR_DC: now also D2.2 (A)
- net PWR_USB: now also D3.2 (A)
- net at R1.2, R2.2: now also JP1.1; no longer C7.1
- net CLKI renamed OSC1
- net OSC1: now also C14.1, R5.1, Y1.3
- net CLKO renamed OSC2
- net OSC2: now also C13.1, R5.2, Y1.1
- new net: C7.1, JP1.2
- new net: D4.1 (K), R7.1
- new net: D2.1 (K), D3.1 (K), R6.1
Other:
- moved on the sheet: C1, C10, C11, C12, C2, C3, C4, C5, C6, C7, C8, C9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

Commit message: inductor
Parts:
- removed D2, D3: LED_B, LED_SMD:LED_0603_1608Metric_Pad1.05x0.95mm_HandSolder, symbol Device:LED_Small
- removed R6: 1.5K, Resistor_SMD:R_0603_1608Metric_Pad0.98x0.95mm_HandSolder, symbol Device:R_Small
- L1: value 8.2u -> 22u; footprint Inductor_SMD:L_Taiyo-Yuden_MD-1616 -> Inductor_SMD:L_Taiyo-Yuden_NR-80xx_HandSoldering
Changed lines of the file:
@@
 P 7450 2050
 F 0 "L1" V 7635 2050 50  0000 C CNN
-F 1 "8.2u" V 7544 2050 50  0000 C CNN
-F 2 "Inductor_SMD:L_Taiyo-Yuden_MD-1616" H 7450 2050 50  0001 C CNN
+F 1 "22u" V 7544 2050 50  0000 C CNN
+F 2 "Inductor_SMD:L_Taiyo-Yuden_NR-80xx_HandSoldering" H 7450 2050 50  0001 C CNN
 F 3 "~" H 7450 2050 50  0001 C CNN
 	1    7450 2050
@@
 Wire Wire Line
 	3200 3500 3200 3650
-Text Label 2000 2700 2    50   ~ 0
-PWR_USB
-Text Label 1550 2700 2    50   ~ 0
-PWR_DC
-Wire Wire Line
-	2000 2950 2000 2700
-Wire Wire Line
-	1550 2950 1550 2700
-Wire Wire Line
-	2000 3550 2000 3650
-Wire Wire Line
-	2000 3250 2000 3350
-Connection ~ 2000 3250
-Wire Wire Line
-	1550 3250 1550 3150
-Wire Wire Line
-	2000 3250 1550 3250
-Wire Wire Line
-	2000 3150 2000 3250
-$Comp
-L power:GND #PWR0128
-U 1 1 60B8F561
-P 2000 3650
-F 0 "#PWR0128" H 2000 3400 50  0001 C CNN
-F 1 "GND" H 2005 3477 50  0000 C CNN
-F 2 "" H 2000 3650 50  0001 C CNN
-F 3 "" H 2000 3650 50  0001 C CNN
-	1    2000 3650
-	1    0    0    -1
-$EndComp
-$Comp
-L Device:R_Small R6
-U 1 1 60B8EA5F
-P 2000 3450
-F 0 "R6" H 2059 3496 50  0000 L CNN
-F 1 "1.5K" H 2059 3405 50  0000 L CNN
-F 2 "Resistor_SMD:R_0603_1608Metric_Pad0.98x0.95mm_HandSolder" H 2000 3450 50  0001 C CNN
-F 3 "~" H 2000 3450 50  0001 C CNN
-	1    2000 3450
-	1    0    0    -1
-$EndComp
-$Comp
-L Device:LED_Small D2
-U 1 1 60B8E4A4
-P 1550 3050
-F 0 "D2" V 1596 2980 50  0000 R CNN
-F 1 "LED_B" V 1505 2980 50  0000 R CNN
-F 2 "LED_SMD:LED_0603_1608Metric_Pad1.05x0.95mm_HandSolder" V 1550 3050 50  0001 C CNN
-F 3 "~" V 1550 3050 50  0001 C CNN
-	1    1550 3050
-	0    -1   -1   0
-$EndComp
-$Comp
-L Device:LED_Small D3
-U 1 1 60B8DE76
-P 2000 3050
-F 0 "D3" V 2046 2980 50  0000 R CNN
-F 1 "LED_B" V 1955 2980 50  0000 R CNN
-F 2 "LED_SMD:LED_0603_1608Metric_Pad1.05x0.95mm_HandSolder" V 2000 3050 50  0001 C CNN
-F 3 "~" V 2000 3050 50  0001 C CNN
-	1    2000 3050
-	0    -1   -1   0
-$EndComp
 $EndSCHEMATC

Commit message: gerber
Connections:
- net AN0: now also J1.19 (Pin_19); no longer J1.13 (Pin_13)
- net AN1: now also J1.22 (Pin_22); no longer J1.14 (Pin_14)
- net GND: now also J1.16 (Pin_16), J1.2 (Pin_2), J1.5 (Pin_5); no longer J1.10 (Pin_10)
- net RA10: now also J1.15 (Pin_15); no longer J1.9 (Pin_9)
- net RA7: now also J1.18 (Pin_18); no longer J1.11 (Pin_11)
- net RB10: now also J1.12 (Pin_12); no longer J1.4 (Pin_4)
- net RB11: now also J1.14 (Pin_14); no longer J1.8 (Pin_8)
- net RB12: now also J1.11 (Pin_11); no longer J1.12 (Pin_12)
- net RB14: now also J1.17 (Pin_17); no longer J1.20 (Pin_20)
- net RB5: now also J5.13 (Pin_13); no longer J1.7 (Pin_7)
- net RB6: now also J5.14 (Pin_14); no longer J1.6 (Pin_6)
- net RB7: now also J1.4 (Pin_4); no longer J5.13 (Pin_13)
- net RC6: now also J1.8 (Pin_8); no longer J1.2 (Pin_2)
- net RC7: now also J1.7 (Pin_7); no longer J1.16 (Pin_16)
- net RC8: now also J1.10 (Pin_10); no longer J1.17 (Pin_17)
- net RC9: now also J1.9 (Pin_9); no longer J1.15 (Pin_15)
- net RB13|U1RX: now reaches U3.2 (TXD)
- net RB13|U1RX: now also J1.13 (Pin_13), U1.11 (RB13)
- net RB15|U1TX: now reaches U3.3 (RXD)
- net RB15|U1TX: now also J1.20 (Pin_20), U1.15 (RB15)
- removed net RB13: J1.5 (Pin_5), U1.11 (RB13)
- removed net RB15: J1.22 (Pin_22), U1.15 (RB15)
- net RB8 renamed RB8|U2RX
- net RB8|U2RX: now also J1.3 (Pin_3); no longer J5.14 (Pin_14)
- net RB9 renamed RB9|U2TX
- net RB9|U2TX: now also J1.6 (Pin_6); no longer J1.3 (Pin_3)
- no-connect marks 3 -> 11
Other:
- moved on the sheet: C1, C10, C11, C12, C13, C14, C15, C16, C17, C18, C2, C3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
