File: PIC32MX150.kicad_sch (KiCad schematic)
At the start: 51 parts, among them J1 GPIO_1, J2 USB_B_Micro, J3 Barrel_Jack, J4 ICSP, J5 GPIO_2, J6 SPI_0, J7 SPI_1, SW1 RST, SW2 SW_SPDT, SW3 SW_SPST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

Commit message: LM22676 active-high
Parts:
- D1: footprint Diode_SMD:D_SMA_Handsoldering -> Diode_SMD:D_SOD-123
Connections:
- net +5V: now also U2.5 (EN)
- net GND: no longer U2.5 (EN)
Other:
- moved on the sheet: C16
Changed lines of the file:
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@@
   (junction (at 142.24 64.77) (diameter 1.016) (color 0 0 0 0))
   (junction (at 151.13 46.99) (diameter 1.016) (color 0 0 0 0))
-  (junction (at 151.13 54.61) (diameter 1.016) (color 0 0 0 0))
   (junction (at 151.13 64.77) (diameter 1.016) (color 0 0 0 0))
+  (junction (at 157.48 46.99) (diameter 1.016) (color 0 0 0 0))
   (junction (at 167.64 64.77) (diameter 1.016) (color 0 0 0 0))
   (junction (at 170.18 104.14) (diameter 1.016) (color 0 0 0 0))
@@
     (stroke (width 0) (type solid) (color 0 0 0 0))
   )
-  (wire (pts (xy 151.13 46.99) (xy 160.02 46.99))
-    (stroke (width 0) (type solid) (color 0 0 0 0))
-  )
-  (wire (pts (xy 151.13 48.26) (xy 151.13 46.99))
-    (stroke (width 0) (type solid) (color 0 0 0 0))
-  )
-  (wire (pts (xy 151.13 53.34) (xy 151.13 54.61))
-    (stroke (width 0) (type solid) (color 0 0 0 0))
-  )
-  (wire (pts (xy 151.13 54.61) (xy 151.13 64.77))
-    (stroke (width 0) (type solid) (color 0 0 0 0))
-  )
-  (wire (pts (xy 151.13 54.61) (xy 160.02 54.61))
+  (wire (pts (xy 151.13 46.99) (xy 157.48 46.99))
+    (stroke (width 0) (type solid) (color 0 0 0 0))
+  )
+  (wire (pts (xy 151.13 53.34) (xy 151.13 46.99))
+    (stroke (width 0) (type solid) (color 0 0 0 0))
+  )
+  (wire (pts (xy 151.13 58.42) (xy 151.13 64.77))
     (stroke (width 0) (type solid) (color 0 0 0 0))
   )
@@
   )
   (wire (pts (xy 153.67 104.14) (xy 153.67 101.6))
+    (stroke (width 0) (type solid) (color 0 0 0 0))
+  )
+  (wire (pts (xy 157.48 46.99) (xy 160.02 46.99))
+    (stroke (width 0) (type solid) (color 0 0 0 0))
+  )
+  (wire (pts (xy 157.48 54.61) (xy 157.48 46.99))
+    (stroke (width 0) (type solid) (color 0 0 0 0))
+  )
+  (wire (pts (xy 160.02 54.61) (xy 157.48 54.61))
     (stroke (width 0) (type solid) (color 0 0 0 0))
   )
@@
       (effects (font (size 1.27 1.27)) (justify left))
     )
-    (property "Footprint" "Diode_SMD:D_SMA_Handsoldering" (id 2) (at 190.5 60.96 90)
+    (property "Footprint" "Diode_SMD:D_SOD-123" (id 2) (at 190.5 60.96 90)
       (effects (font (size 1.27 1.27)) hide)
     )
@@
     (pin "2")
   )
-  (symbol (lib_id "PIC32MX150-rescue:C_Small-Device") (at 151.13 50.8 0) (unit 1)
-    (in_bom yes) (on_board yes)
-    (property "Reference" "C16" (id 0) (at 153.4668 49.6316 0)
-      (effects (font (size 1.27 1.27)) (justify left))
-    )
-    (property "Value" "100n" (id 1) (at 153.4668 51.943 0)
-      (effects (font (size 1.27 1.27)) (justify left))
-    )
-    (property "Footprint" "Capacitor_SMD:C_0603_1608Metric_Pad1.08x0.95mm_HandSolder" (id 2) (at 151.13 50.8 0)
-      (effects (font (size 1.27 1.27)) hide)
-    )
-    (property "Datasheet" "~" (id 3) (at 151.13 50.8 0)
+  (symbol (lib_id "PIC32MX150-rescue:C_Small-Device") (at 151.13 55.88 0) (unit 1)
+    (in_bom yes) (on_board yes)
+    (property "Reference" "C16" (id 0) (at 153.4668 54.7116 0)
+      (effects (font (size 1.27 1.27)) (justify left))
+    )
+    (property "Value" "100n" (id 1) (at 153.4668 57.023 0)
+      (effects (font (size 1.27 1.27)) (justify left))
+    )
+    (property "Footprint" "Capacitor_SMD:C_0603_1608Metric_Pad1.08x0.95mm_HandSolder" (id 2) (at 151.13 55.88 0)
+      (effects (font (size 1.27 1.27)) hide)
+    )
+    (property "Datasheet" "~" (id 3) (at 151.13 55.88 0)
       (effects (font (size 1.27 1.27)) hide)
     )
@@
     )
     (path "/00000000-0000-0000-0000-00006072f91f"
-      (reference "D1") (unit 1) (value "EJ1S") (footprint "Diode_SMD:D_SMA_Handsoldering")
+      (reference "D1") (unit 1) (value "EJ1S") (footprint "Diode_SMD:D_SOD-123")
     )
     (path "/715a5923-0e0d-414a-be07-857020fe033d"
